Commit message: added urdf meshes for G1

File: g1/sim/G1_rviz_simulation-main/G1_rviz_simulation-main/urdf/g1_29dof_with_hand_rev_1_0_pkg.urdf (robot description, URDF)
Before this commit: robot g1_29dof_with_hand_rev_1_0, 53 links, 52 joints
Links:
- added link base_link
Joints:
- added joint base_link_to_pelvis: type fixed, parent base_link, child pelvis
